File: vogelhuisje_kicad/Power_supply.sch (KiCad schematic (older format))
At the start: 0 parts

Commit message: Update ESP_arduino.sch-bak, Power_supply.sch, and 25 more files...
Parts:
- added D1: D_Zener, Diode_SMD:D_SMB_Handsoldering, symbol Device:D_Zener
- added J1: Conn_01x02, Connector_JST:JST_PH_B2B-PH-K_1x02_P2.00mm_Vertical, symbol Connector_Generic:Conn_01x02
- added J2: Conn_01x02_Female, Connector_PinSocket_2.54mm:PinSocket_1x02_P2.54mm_Vertical, symbol Connector:Conn_01x02_Female
- added J3: USB_C_Receptacle_USB2.0, Connector_USB:USB_C_Receptacle_HRO_TYPE-C-31-M-12, symbol Connector:USB_C_Receptacle_USB2.0
- added P1: TP4056breakout, Components:TP4056breakout, symbol TP4056-breakout:TP4056breakout
- added P2: GenericBoostConverter, Components:GenericBoostConverter, symbol TP4056-breakout:GenericBoostConverter
- added Q1: Q_PMOS_GSD, Package_TO_SOT_SMD:SOT-23, symbol Device:Q_PMOS_GSD
- added R1: 100k, Resistor_THT:R_Axial_DIN0207_L6.3mm_D2.5mm_P7.62mm_Horizontal, symbol Device:R
Connections:
- new net: D1.2 (A), J2.2 (Pin_2), P1.1 (Vin+), Q1.1 (G), R1.1
- new net: J1.1 (Pin_1), P1.3 (OUT+), P1.4 (B+), Q1.3 (D)
- new net: J1.2 (Pin_2), P1.5 (B-)
- new net: D1.1 (K), P2.1 (Vin+), Q1.2 (S)
- new net 5V: J3.A4 (VBUS), J3.A9 (VBUS), J3.B4 (VBUS), J3.B9 (VBUS), P2.3 (Vout+)
- new net GND: J2.1 (Pin_1), J3.A1 (GND), J3.A12 (GND), J3.B1 (GND), J3.B12 (GND), J3.S1 (SHIELD), P1.2 (GND), P1.6 (OUT-), P2.2 (GND), P2.4 (GND), R1.2
Changed lines of the file:
@@
 $Descr A4 11693 8268
 encoding utf-8
-Sheet 1 3
+Sheet 2 3
 Title ""
 Date ""
@@
 Comment4 ""
 $EndDescr
+$Comp
+L TP4056-breakout:TP4056breakout P1
+U 1 1 6263DE48
+P 2550 2300
+F 0 "P1" H 2575 2825 50  0000 C CNN
+F 1 "TP4056breakout" H 2575 2734 50  0000 C CNN
+F 2 "Components:TP4056breakout" H 2500 2700 50  0001 C CNN
+F 3 "" H 2500 2700 50  0001 C CNN
+	1    2550 2300
+	1    0    0    -1
+$EndComp
+$Comp
+L TP4056-breakout:GenericBoostConverter P2
+U 1 1 6263E192
+P 5450 2300
+F 0 "P2" H 5450 2715 50  0000 C CNN
+F 1 "GenericBoostConverter" H 5450 2624 50  0000 C CNN
+F 2 "Components:GenericBoostConverter" H 5450 2450 50  0001 C CNN
+F 3 "" H 5450 2450 50  0001 C CNN
+	1    5450 2300
+	1    0    0    -1
+$EndComp
+$Comp
+L Device:R R1
+U 1 1 6263EAD6
+P 3600 2250
+F 0 "R1" H 3670 2296 50  0000 L CNN
+F 1 "100k" H 3670 2205 50  0000 L CNN
+F 2 "Resistor_THT:R_Axial_DIN0207_L6.3mm_D2.5mm_P7.62mm_Horizontal" V 3530 2250 50  0001 C CNN
+F 3 "~" H 3600 2250 50  0001 C CNN
+	1    3600 2250
+	1    0    0    -1
+$EndComp
+Wire Wire Line
+	3600 2100 3600 1750
+Wire Wire Line
+	1950 1750 1950 2050
+$Comp
+L power:GND #PWR0101
+U 1 1 6263EF5E
+P 1950 2400
+F 0 "#PWR0101" H 1950 2150 50  0001 C CNN
+F 1 "GND" H 1955 2227 50  0000 C CNN
+F 2 "" H 1950 2400 50  0001 C CNN
+F 3 "" H 1950 2400 50  0001 C CNN
+	1    1950 2400
+	1    0    0    -1
+$EndComp
+Wire Wire Line
+	3350 1400 3350 2300
+Wire Wire Line
+	3350 2300 3200 2300
+Wire Wire Line
+	3200 2450 3600 2450
+Wire Wire Line
+	3600 2450 3600 2400
+Connection ~ 3600 2450
+Wire Wire Line
+	3600 1750 3850 1750
+Wire Wire Line
+	4200 1950 4200 2150
+Wire Wire Line
+	4200 2150 4850 2150
+$Comp
+L Device:D_Zener D1
+U 1 1 62643FC2
+P 3850 1900
+F 0 "D1" V 3896 1821 50  0000 R CNN
+F 1 "D_Zener" V 3805 1821 50  0000 R CNN
+F 2 "Diode_SMD:D_SMB_Handsoldering" H 3850 1900 50  0001 C CNN
+F 3 "~" H 3850 1900 50  0001 C CNN
+	1    3850 1900
+	0    -1   -1   0
+$EndComp
+Connection ~ 3850 1750
+Wire Wire Line
+	3850 1750 3900 1750
+Wire Wire Line
+	3850 2050 3850 2150
+Wire Wire Line
+	3850 2150 4200 2150
+Connection ~ 4200 2150
+$Comp
+L Connector_Generic:Conn_01x02 J1
+U 1 1 62647C4D
+P 3250 1200
+F 0 "J1" H 3168 875 50  0000 C CNN
+F 1 "Conn_01x02" H 3168 966 50  0000 C CNN
+F 2 "Connector_JST:JST_PH_B2B-PH-K_1x02_P2.00mm_Vertical" H 3250 1200 50  0001 C CNN
+F 3 "~" H 3250 1200 50  0001 C CNN
+	1    3250 1200
+	0    -1   -1   0
+$EndComp
+Wire Wire Line
+	3200 2150 3250 2150
+Wire Wire Line
+	3200 2000 3250 2000
+Connection ~ 3250 2000
+Wire Wire Line
+	3250 2000 3250 1550
+Wire Wire Line
+	3600 1750 1950 1750
+Connection ~ 3600 1750
+Wire Wire Line
+	3250 2000 3250 2150
+Wire Wire Line
+	4200 1550 3250 1550
+Connection ~ 3250 1550
+Wire Wire Line
+	3250 1550 3250 1400
+$Comp
+L Device:Q_PMOS_GSD Q1
+U 1 1 6264EDFF
+P 4100 1750
+F 0 "Q1" H 4305 1796 50  0000 L CNN
+F 1 "Q_PMOS_GSD" H 4305 1705 50  0000 L CNN
+F 2 "Package_TO_SOT_SMD:SOT-23" H 4300 1850 50  0001 C CNN
+F 3 "~" H 4100 1750 50  0001 C CNN
+	1    4100 1750
+	1    0    0    -1
+$EndComp
+$Comp
+L Connector:USB_C_Receptacle_USB2.0 J3
+U 1 1 62654366
+P 5100 3300
+F 0 "J3" V 5253 4029 50  0000 L CNN
+F 1 "USB_C_Receptacle_USB2.0" V 5162 4029 50  0000 L CNN
+F 2 "Connector_USB:USB_C_Receptacle_HRO_TYPE-C-31-M-12" H 5250 3300 50  0001 C CNN
+F 3 "https://www.usb.org/sites/default/files/documents/usb_type-c.zip" H 5250 3300 50  0001 C CNN
+	1    5100 3300
+	0    -1   -1   0
+$EndComp
+Wire Wire Line
+	4500 2700 4500 2600
+Wire Wire Line
+	4500 2600 6100 2600
+Wire Wire Line
+	6100 2600 6100 2150
+Wire Wire Line
+	6100 2150 6050 2150
+Wire Wire Line
+	6050 2450 6050 3300
+Wire Wire Line
+	6050 3300 6000 3300
+Wire Wire Line
+	6050 3300 6050 3600
+Wire Wire Line
+	6050 3600 6000 3600
+Connection ~ 6050 3300
+Text HLabel 6300 2150 2    50   Input ~ 0
+5V
+Wire Wire Line
+	6100 2150 6300 2150
+Connection ~ 6100 2150
+Wire Wire Line
+	3600 2450 4850 2450
+Connection ~ 6050 2450
+Wire Wire Line
+	6050 2450 6200 2450
+$Comp
+L Connector:Conn_01x02_Female J2
+U 1 1 62641E6A
+P 1650 2250
+F 0 "J2" H 1542 1925 50  0000 C CNN
+F 1 "Conn_01x02_Female" H 1542 2016 50  0000 C CNN
+F 2 "Connector_PinSocket_2.54mm:PinSocket_1x02_P2.54mm_Vertical" H 1650 2250 50  0001 C CNN
+F 3 "~" H 1650 2250 50  0001 C CNN
+	1    1650 2250
+	-1   0    0    1
+$EndComp
+Wire Wire Line
+	1850 2250 1950 2250
+Wire Wire Line
+	1950 2250 1950 2400
+Connection ~ 1950 2400
+Wire Wire Line
+	1850 2150 1950 2150
+Wire Wire Line
+	1950 2150 1950 2050
+Connection ~ 1950 2050
+$Comp
+L power:GND #PWR0102
+U 1 1 62647069
+P 3600 2450
+F 0 "#PWR0102" H 3600 2200 50  0001 C CNN
+F 1 "GND" H 3605 2277 50  0000 C CNN
+F 2 "" H 3600 2450 50  0001 C CNN
+F 3 "" H 3600 2450 50  0001 C CNN
+	1    3600 2450
+	1    0    0    -1
+$EndComp
+$Comp
+L power:GND #PWR0103
+U 1 1 626475C4
+P 6200 2450
+F 0 "#PWR0103" H 6200 2200 50  0001 C CNN
+F 1 "GND" H 6205 2277 50  0000 C CNN
+F 2 "" H 6200 2450 50  0001 C CNN
+F 3 "" H 6200 2450 50  0001 C CNN
+	1    6200 2450
+	1    0    0    -1
+$EndComp
+Connection ~ 6200 2450
+Wire Wire Line
+	6200 2450 6300 2450
+Text HLabel 6300 2450 2    50   Input ~ 0
+GND
 $EndSCHEMATC
