File: vogelhuisje_kicad/_autosave-vogelhuisje_kicad.sch (KiCad schematic (older format))
At the start: 0 parts

Commit message: Update ESP_arduino.sch-bak, Power_supply.sch, and 25 more files...
Changed lines of the file:
@@
 $EndDescr
 $Sheet
-S 1850 1800 2700 2400
+S 1700 2300 1300 850
 U 6263B8AD
 F0 "Power Supply" 50
 F1 "Power_supply.sch" 50
-F2 "5V" I R 4550 2700 50
+F2 "5V" I R 3000 2550 50
+F3 "GND" I R 3000 2850 50
 $EndSheet
 $Sheet
