File: vogelhuisje_kicad/Camera_module.sch (KiCad schematic (older format))
At the start: 11 parts, among them U1 XC6206-2.8V, U2 XC6206-1.2V

Commit message: Update Camera_module.sch, Camera_module.sch-bak, and 5 more files...
Parts:
- added D? (x4): LED, symbol Device:LED
- added Q?: Q_NMOS_DSG, symbol Device:Q_NMOS_DSG
- added R? (x2): R, symbol Device:R
Connections:
- net GND: now also Q?.1 (D)
- new net: Q?.3 (G), R?.2
- new net: D?.1 (K), D?.1 (K), Q?.2 (S)
- new net: D?.1 (K), D?.1 (K), D?.2 (A), D?.2 (A)
- new net: D?.2 (A), D?.2 (A), R?.2
- new net V_led_switch-: R?.1
- new net Vbat: R?.1
Changed lines of the file:
@@
 	6250 2550 6250 2950
 Connection ~ 6250 2950
+Text HLabel 9450 4100 2    50   Input ~ 0
+V_led_switch-
+Text HLabel 8800 2450 2    50   Input ~ 0
+Vbat
+$Comp
+L Device:R R?
+U 1 1 626DA198
+P 9250 4100
+F 0 "R?" V 9043 4100 50  0000 C CNN
+F 1 "R" V 9134 4100 50  0000 C CNN
+F 2 "" V 9180 4100 50  0001 C CNN
+F 3 "~" H 9250 4100 50  0001 C CNN
+	1    9250 4100
+	0    1    1    0
+$EndComp
+$Comp
+L Device:Q_NMOS_DSG Q?
+U 1 1 626DDEE8
+P 8900 4100
+F 0 "Q?" H 9105 4054 50  0000 L CNN
+F 1 "Q_NMOS_DSG" H 9105 4145 50  0000 L CNN
+F 2 "" H 9100 4200 50  0001 C CNN
+F 3 "~" H 8900 4100 50  0001 C CNN
+	1    8900 4100
+	-1   0    0    1
+$EndComp
+Wire Wire Line
+	9400 4100 9450 4100
+$Comp
+L power:GND #PWR?
+U 1 1 626E602C
+P 8800 4300
+F 0 "#PWR?" H 8800 4050 50  0001 C CNN
+F 1 "GND" H 8805 4127 50  0000 C CNN
+F 2 "" H 8800 4300 50  0001 C CNN
+F 3 "" H 8800 4300 50  0001 C CNN
+	1    8800 4300
+	1    0    0    -1
+$EndComp
+$Comp
+L Device:LED D?
+U 1 1 626E6646
+P 8650 3450
+F 0 "D?" V 8689 3333 50  0000 R CNN
+F 1 "LED" V 8598 3333 50  0000 R CNN
+F 2 "" H 8650 3450 50  0001 C CNN
+F 3 "~" H 8650 3450 50  0001 C CNN
+	1    8650 3450
+	0    -1   -1   0
+$EndComp
+$Comp
+L Device:LED D?
+U 1 1 626E73B6
+P 8950 3450
+F 0 "D?" V 8989 3333 50  0000 R CNN
+F 1 "LED" V 8898 3333 50  0000 R CNN
+F 2 "" H 8950 3450 50  0001 C CNN
+F 3 "~" H 8950 3450 50  0001 C CNN
+	1    8950 3450
+	0    -1   -1   0
+$EndComp
+$Comp
+L Device:LED D?
+U 1 1 626E8633
+P 8650 3100
+F 0 "D?" V 8689 2983 50  0000 R CNN
+F 1 "LED" V 8598 2983 50  0000 R CNN
+F 2 "" H 8650 3100 50  0001 C CNN
+F 3 "~" H 8650 3100 50  0001 C CNN
+	1    8650 3100
+	0    -1   -1   0
+$EndComp
+$Comp
+L Device:LED D?
+U 1 1 626E9899
+P 8950 3100
+F 0 "D?" V 8989 2983 50  0000 R CNN
+F 1 "LED" V 8898 2983 50  0000 R CNN
+F 2 "" H 8950 3100 50  0001 C CNN
+F 3 "~" H 8950 3100 50  0001 C CNN
+	1    8950 3100
+	0    -1   -1   0
+$EndComp
+Wire Wire Line
+	8950 3250 8950 3300
+Wire Wire Line
+	8950 3250 8650 3250
+Connection ~ 8950 3250
+Wire Wire Line
+	8650 3300 8650 3250
+Connection ~ 8650 3250
+Wire Wire Line
+	8650 3600 8650 3750
+Wire Wire Line
+	8650 3750 8800 3750
+Wire Wire Line
+	8950 3750 8950 3600
+Wire Wire Line
+	8800 3900 8800 3750
+Connection ~ 8800 3750
+Wire Wire Line
+	8800 3750 8950 3750
+Wire Wire Line
+	8650 2950 8650 2900
+Wire Wire Line
+	8650 2900 8800 2900
+Wire Wire Line
+	8950 2900 8950 2950
+$Comp
+L Device:R R?
+U 1 1 626F28F9
+P 8800 2700
+F 0 "R?" H 8870 2746 50  0000 L CNN
+F 1 "R" H 8870 2655 50  0000 L CNN
+F 2 "" V 8730 2700 50  0001 C CNN
+F 3 "~" H 8800 2700 50  0001 C CNN
+	1    8800 2700
+	1    0    0    -1
+$EndComp
+Wire Wire Line
+	8800 2450 8800 2550
+Wire Wire Line
+	8800 2850 8800 2900
+Connection ~ 8800 2900
+Wire Wire Line
+	8800 2900 8950 2900
 $EndSCHEMATC
