File: vogelhuisje_kicad/vogelhuisje_kicad.kicad_pcb (KiCad board)
At the start: 2 copper layers, 8 parts, among them J1 Conn_01x02, J2 Conn_01x02_Female, J3 USB_C_Receptacle_USB2.0, P1 TP4056breakout, P2 GenericBoostConverter, Q1 Q_PMOS_GSD

Commit message: PCB design
Parts:
- added A1: Arduino_Nano_v3.x, Module:Arduino_Nano, F.Cu at (101.8, 164.9)
- added D1: D_Schottky, Diode_SMD:D_SMB_Handsoldering, F.Cu at (85.0, 72.0)
- added D2: D, Diode_THT:D_5W_P12.70mm_Horizontal, F.Cu at (95.0, 76.7)
- added J6: Conn_01x19_Female, Connector_PinHeader_2.54mm:PinHeader_1x19_P2.54mm_Vertical, F.Cu at (151.0, 117.0)
- added U3: ESP32-LilyGo-T_PCIE, components:Lilygo_T_PCIE, F.Cu at (113.8, 125.5)
- added U4: PMS5003, Connector_PinSocket_2.54mm:PinSocket_1x08_P2.54mm_Vertical, F.Cu at (117.3, 171.8)
- added U5: SD-card-reader, Connector_PinSocket_2.54mm:PinSocket_1x06_P2.54mm_Vertical, F.Cu at (126.8, 172.2)
- added U6: BME280Breakout, Connector_PinHeader_2.54mm:PinHeader_1x06_P2.54mm_Vertical, F.Cu at (112.2, 178.2)
- added U7: BME280Breakout, Connector_PinHeader_2.54mm:PinHeader_1x06_P2.54mm_Vertical, F.Cu at (133.6, 178.4)
- D1: value D_Zener -> D_Schottky
- J3: footprint Connector_USB:USB_C_Receptacle_HRO_TYPE-C-31-M-12 -> components:GCT_USB4125-GF-A-0190_REVA2
- renumbered J2 to J1, J1 to J2, R1 to R2
Connections:
- net Net-(J1-Pad1) renamed /Power Supply/Vbat
- J3 pad A5: Net-(J3-PadA5) -> unconnected-(J3-PadA5)
- J3 pad A9: /Power Supply/5V -> +5V
- J3 pad B5: Net-(J3-PadB5) -> unconnected-(J3-PadB5)
- J3 pad B9: /Power Supply/5V -> +5V
- P1 pad 6: GND -> Net-(P1-Pad6)
- P2 pad 2: GND -> Net-(P1-Pad6)
- P2 pad 3: /Power Supply/5V -> +5V
- Q1 pad 1: Net-(D1-Pad2) -> Net-(D2-Pad1)
- R2 pad 2: GND -> Net-(P1-Pad6)
Routing:
- net +5V: track 0.00 -> 57.8 mm, vias 0 -> 1
- net /Power Supply/5V: track 57.7 -> 0.00 mm, vias 1 -> 0
- net GND: track 99.5 -> 72.7 mm
- net Net-(D1-Pad2): track 52.7 -> 38.4 mm
- net Net-(D2-Pad1): track 0.00 -> 0.70 mm
Other:
- net class Default removed
- rule pad_to_mask_clearance: 0.051 -> 0
- rule solder_mask_min_width: 0.25 -> 0.12

Commit message: PCB done with version 1
Parts:
- removed the D1 at (85.0, 72.0)
- added ?: , , F.Cu at (150.0, 75.0)
- added ?: , , F.Cu at (70.0, 175.0)
- added ?: , , F.Cu at (150.0, 175.0)
- added R1: -, Resistor_THT:R_Axial_DIN0207_L6.3mm_D2.5mm_P7.62mm_Horizontal, F.Cu at (80.0, 162.8)
- added REF**: MountingHole_4.3mm_M4_ISO7380_Pad, MountingHole:MountingHole_4.3mm_M4_ISO7380_Pad, F.Cu at (70.0, 74.0)
- moved U6 31.5 mm to (143.3, 174.0)
- moved U5 15.8 mm to (111.1, 170.0)
- moved A1 14.0 mm to (87.9, 162.8)
- moved U4 13.4 mm to (104.0, 170.1)
- moved U7 13.0 mm to (143.5, 170.0)
Connections:
- P1 pad 6: Net-(P1-Pad6) -> GND
- P2 pad 2: Net-(P1-Pad6) -> GND
- R2 pad 2: Net-(P1-Pad6) -> GND
- U3 pad 17: Net-(U3-Pad17) -> GND
- U6 pad 2: Net-(U3-Pad17) -> GND
- U7 pad 2: Net-(U3-Pad17) -> GND
Routing:
- net /Power Supply/Vbat: track 18.5 -> 148.5 mm
- net +5V: track 57.8 -> 185.5 mm, vias 1 -> 2
- net Net-(D2-Pad1): track 0.70 -> 102.8 mm, vias 0 -> 3
- net +3V3: track 0.00 -> 97.8 mm
- net GND: track 72.7 -> 0.73 mm, vias 0 -> 2
- net /Sensors and microcontrollers/PCLK_CAM: track 0.00 -> 66.3 mm, vias 0 -> 2
- net Net-(U3-Pad16): track 0.00 -> 64.5 mm, vias 0 -> 1
- net /Sensors and microcontrollers/XCLK_CAM: track 0.00 -> 63.5 mm, vias 0 -> 1
- net /Sensors and microcontrollers/TX_ARD: track 0.00 -> 60.3 mm, vias 0 -> 2
- net /Sensors and microcontrollers/RX_ARD: track 0.00 -> 59.9 mm
- net /Sensors and microcontrollers/LED_EN: track 0.00 -> 58.8 mm, vias 0 -> 1
- net /Sensors and microcontrollers/Y6_CAM: track 0.00 -> 55.1 mm
- net /Sensors and microcontrollers/SCL: track 0.00 -> 53.5 mm, vias 0 -> 1
- net /Sensors and microcontrollers/INT_OUT_ARD: track 0.00 -> 51.4 mm
- net /Sensors and microcontrollers/HREF_CAM: track 0.00 -> 51.1 mm, vias 0 -> 2
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- added copper zone on B.Cu, net GND
- added copper zone on F.Cu, net GND
Other:
- board outline added: 95 x 115 mm
