File: vogelhuisje_kicad/ESP_arduino.kicad_sch (KiCad schematic)
At the start: 6 parts, among them U3 ESP32-LilyGo-T_PCIE, U4 PMS5003, U5 SD-card-reader, U6 BME280Breakout, U7 BME280Breakout

Commit message: PCB done with version 1
Connections:
- net GND: now also U3.17 (GND), U6.2 (GND), U7.2 (GND)
Changed lines of the file:
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@@
     (pin "8")
+  )
+  (symbol (lib_id "power:GND") (at 146.05 132.08 0) (unit 1)
+    (in_bom yes) (on_board yes) (fields_autoplaced)
+    (property "Reference" "#PWR?" (id 0) (at 146.05 138.43 0)
+      (effects (font (size 1.27 1.27)) hide)
+    )
+    (property "Value" "GND" (id 1) (at 146.05 137.16 0))
+    (property "Footprint" "" (id 2) (at 146.05 132.08 0)
+      (effects (font (size 1.27 1.27)) hide)
+    )
+    (property "Datasheet" "" (id 3) (at 146.05 132.08 0)
+      (effects (font (size 1.27 1.27)) hide)
+    )
+    (pin "1")
   )
   (symbol (lib_id "power:GND") (at 140.97 64.77 0) (unit 1)

Commit message: Kicad Changes Tadjiro
Board now supports 3 lipo cells and a motion sensor.
Connections:
- net Motion_out: now reaches A1.22 (A3)
- no-connect marks 30 -> 27
Changed lines of the file:
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@@
   (no_connect (at 88.9 151.13))
   (no_connect (at 88.9 146.05))
-  (no_connect (at 88.9 143.51))
   (no_connect (at 127 165.1))
   (no_connect (at 127 167.64))
   (no_connect (at 127 170.18))
   (no_connect (at 127 172.72))
-  (no_connect (at 87.63 39.37))
   (no_connect (at 113.03 46.99))
-  (no_connect (at 113.03 49.53))
   (no_connect (at 113.03 59.69))
   (no_connect (at 113.03 57.15))
@@
     (stroke (width 0) (type default) (color 0 0 0 0))
   )
-  (wire (pts (xy 80.01 80.01) (xy 80.01 15.24))
-    (stroke (width 0) (type default) (color 0 0 0 0))
-  )
   (wire (pts (xy 54.61 60.96) (xy 54.61 62.23))
     (stroke (width 0) (type default) (color 0 0 0 0))
@@
     (stroke (width 0) (type default) (color 0 0 0 0))
   )
-  (wire (pts (xy 50.8 140.97) (xy 68.58 140.97))
+  (wire (pts (xy 80.01 15.24) (xy 80.01 80.01))
+    (stroke (width 0) (type default) (color 0 0 0 0))
+  )
+  (wire (pts (xy 50.8 144.78) (xy 68.58 140.97))
     (stroke (width 0) (type default) (color 0 0 0 0))
   )
@@
     (effects (font (size 1.27 1.27)) (justify right bottom))
   )
+  (label "Motion_out" (at 50.8 140.97 0)
+    (effects (font (size 1.27 1.27)) (justify left bottom))
+  )
   (label "HREF_CAM" (at 88.9 133.35 180)
     (effects (font (size 1.27 1.27)) (justify right bottom))
@@
     (effects (font (size 1.27 1.27)) (justify left bottom))
   )
+  (label "Motion_out" (at 113.03 49.53 0)
+    (effects (font (size 1.27 1.27)) (justify left bottom))
+  )
   (label "PWDN_CAM" (at 81.28 97.79 0)
     (effects (font (size 1.27 1.27)) (justify left bottom))
@@
     (effects (font (size 1.27 1.27)) (justify left bottom))
   )
-  (hierarchical_label "3V3" (shape input) (at 50.8 140.97 180)
+  (hierarchical_label "3V3" (shape input) (at 50.8 144.78 180)
     (effects (font (size 1.27 1.27)) (justify right))
   )
@@
   )
   (hierarchical_label "Vbat" (shape input) (at 50.8 80.01 180)
+    (effects (font (size 1.27 1.27)) (justify right))
+  )
+  (hierarchical_label "Motion_out" (shape input) (at 50.8 140.97 180)
     (effects (font (size 1.27 1.27)) (justify right))
   )
@@
   (symbol (lib_id "power:GND") (at 146.05 132.08 0) (unit 1)
     (in_bom yes) (on_board yes) (fields_autoplaced)
-    (property "Reference" "#PWR?" (id 0) (at 146.05 138.43 0)
-      (effects (font (size 1.27 1.27)) hide)
-    )
+    (property "Reference" "#PWR0105" (id 0) (at 146.05 138.43 0)
+      (effects (font (size 1.27 1.27)) hide)
+    )
