File: vogelhuisje_camera_board/vogelhuisje_camera_board/vogelhuisje_camera_board.kicad_pcb (KiCad board)
At the start: 2 copper layers, 30 x 84 mm, 19 parts, among them J1 Conn_01x19_Female, J4 Camera Connector, Q2 Q_NMOS_DSG, U1 XC6206-2.8V, U2 XC6206-1.2V

Commit message: PCB done with version 1
Parts:
- added REF**: MountingHole_2.2mm_M2, MountingHole:MountingHole_2.2mm_M2, F.Cu at (92.5, 72.5)
- added REF**: MountingHole_2.2mm_M2, MountingHole:MountingHole_2.2mm_M2, F.Cu at (92.5, 147.5)
- added REF**: MountingHole_2.2mm_M2, MountingHole:MountingHole_2.2mm_M2, F.Cu at (127.5, 72.5)
- added REF**: MountingHole_2.2mm_M2, MountingHole:MountingHole_2.2mm_M2, F.Cu at (127.5, 147.5)
Other:
- board size 30 x 84 mm -> 40 x 84 mm
