File: vogelhuisje_camera_board/vogelhuisje_camera_board/Camera_module.kicad_sch (KiCad schematic)
At the start: 17 parts, among them J4 Camera Connector, Q2 Q_NMOS_DGS

Commit message: Old changes reuploaded
Weird thing happened with git pushes. Hopefully this will solve the problems
Parts:
- added R100k2, R100k3: 100kOhm, Resistor_THT:R_Axial_DIN0207_L6.3mm_D2.5mm_P10.16mm_Horizontal, symbol Device:R
Connections:
- net CSI_1.2V: now also R100k3.1
- net CSI_2.8V: now also R100k2.1
- net GND: now also R100k2.2, R100k3.2
Changed lines of the file:
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@@
   (junction (at 182.88 74.93) (diameter 0) (color 0 0 0 0)
   )
+  (junction (at 181.61 104.14) (diameter 0) (color 0 0 0 0)
+  )
   (junction (at 158.75 96.52) (diameter 0) (color 0 0 0 0)
   )
   (junction (at 111.76 106.68) (diameter 0) (color 0 0 0 0)
   )
+  (junction (at 189.23 96.52) (diameter 0) (color 0 0 0 0)
+  )
   (junction (at 158.75 85.09) (diameter 0) (color 0 0 0 0)
   )
@@
   (junction (at 123.19 101.6) (diameter 0) (color 0 0 0 0)
   )
+  (junction (at 189.23 74.93) (diameter 0) (color 0 0 0 0)
+  )
   (junction (at 223.52 95.25) (diameter 0) (color 0 0 0 0)
   )
   (junction (at 181.61 96.52) (diameter 0) (color 0 0 0 0)
+  )
+  (junction (at 182.88 82.55) (diameter 0) (color 0 0 0 0)
   )
   (junction (at 219.71 82.55) (diameter 0) (color 0 0 0 0)
@@
   (no_connect (at 101.6 121.92))
   (no_connect (at 100.33 66.04))
+  (wire (pts (xy 182.88 82.55) (xy 189.23 82.55))
+    (stroke (width 0) (type default) (color 0 0 0 0))
+  )
   (wire (pts (xy 158.75 104.14) (xy 168.91 104.14))
     (stroke (width 0) (type default) (color 0 0 0 0))
@@
     (stroke (width 0) (type default) (color 0 0 0 0))
   )
-  (wire (pts (xy 182.88 74.93) (xy 191.77 74.93))
+  (wire (pts (xy 182.88 74.93) (xy 189.23 74.93))
     (stroke (width 0) (type default) (color 0 0 0 0))
   )
@@
     (stroke (width 0) (type default) (color 0 0 0 0))
   )
+  (wire (pts (xy 181.61 104.14) (xy 189.23 104.14))
+    (stroke (width 0) (type default) (color 0 0 0 0))
+  )
   (wire (pts (xy 219.71 91.44) (xy 219.71 95.25))
     (stroke (width 0) (type default) (color 0 0 0 0))
@@
     (stroke (width 0) (type default) (color 0 0 0 0))
   )
-  (wire (pts (xy 181.61 96.52) (xy 190.5 96.52))
-    (stroke (width 0) (type default) (color 0 0 0 0))
-  )
   (wire (pts (xy 111.76 110.49) (xy 114.3 110.49))
     (stroke (width 0) (type default) (color 0 0 0 0))
@@
     (stroke (width 0) (type default) (color 0 0 0 0))
   )
+  (wire (pts (xy 189.23 74.93) (xy 191.77 74.93))
+    (stroke (width 0) (type default) (color 0 0 0 0))
+  )
   (wire (pts (xy 158.75 74.93) (xy 161.29 74.93))
     (stroke (width 0) (type default) (color 0 0 0 0))
@@
     (stroke (width 0) (type default) (color 0 0 0 0))
   )
+  (wire (pts (xy 181.61 96.52) (xy 189.23 96.52))
+    (stroke (width 0) (type default) (color 0 0 0 0))
+  )
   (wire (pts (xy 96.52 93.98) (xy 100.33 93.98))
     (stroke (width 0) (type default) (color 0 0 0 0))
@@
   )
   (wire (pts (xy 227.33 73.66) (xy 227.33 74.93))
+    (stroke (width 0) (type default) (color 0 0 0 0))
+  )
+  (wire (pts (xy 189.23 96.52) (xy 190.5 96.52))
     (stroke (width 0) (type default) (color 0 0 0 0))
   )
@@
       (effects (font (size 1.27 1.27)) hide)
     )
+    (pin "1")
+    (pin "2")
+  )
+  (symbol (lib_id "Device:R") (at 189.23 100.33 0) (unit 1)
+    (in_bom yes) (on_board yes)
+    (property "Reference" "R100k3" (id 0) (at 191.008 99.1616 0)
+      (effects (font (size 1.27 1.27)) (justify left))
+    )
+    (property "Value" "100kOhm" (id 1) (at 191.008 101.473 0)
+      (effects (font (size 1.27 1.27)) (justify left))
+    )
+    (property "Footprint" "Resistor_THT:R_Axial_DIN0207_L6.3mm_D2.5mm_P10.16mm_Horizontal" (id 2) (at 187.452 100.33 90)
+      (effects (font (size 1.27 1.27)) hide)
+    )
+    (property "Datasheet" "~" (id 3) (at 189.23 100.33 0)
+      (effects (font (size 1.27 1.27)) hide)
+    )
+    (pin "1")
+    (pin "2")
+  )
+  (symbol (lib_id "Device:R") (at 189.23 78.74 0) (unit 1)
+    (in_bom yes) (on_board yes)
+    (property "Reference" "R100k2" (id 0) (at 191.008 77.5716 0)
+      (effects (font (size 1.27 1.27)) (justify left))
+    )
+    (property "Value" "100kOhm" (id 1) (at 191.008 79.883 0)
+      (effects (font (size 1.27 1.27)) (justify left))
+    )
+    (property "Footprint" "Resistor_THT:R_Axial_DIN0207_L6.3mm_D2.5mm_P10.16mm_Horizontal" (id 2) (at 187.452 78.74 90)
+      (effects (font (size 1.27 1.27)) hide)
+    )
+    (property "Datasheet" "~" (id 3) (at 189.23 78.74 0)
+      (effects (font (size 1.27 1.27)) hide)
+    )
