File: vogelhuisje_camera_board/vogelhuisje_camera_board/Camera_module.kicad_sch (KiCad schematic)
At the start: 19 parts, among them J4 Camera Connector, Q2 Q_NMOS_DGS

Commit message: forgot to save
Parts:
- URegulator1.2, URegulator2.8: footprint Package_TO_SOT_SMD:SOT-23-3 -> Package_TO_SOT_THT:TO-92
Changed lines of the file:
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@@
     (property "Reference" "URegulator2.8" (id 0) (at 168.91 68.7832 0))
     (property "Value" "2.8V regulator" (id 1) (at 168.91 71.0946 0))
-    (property "Footprint" "Package_TO_SOT_SMD:SOT-23-3" (id 2) (at 168.91 69.215 0)
+    (property "Footprint" "Package_TO_SOT_THT:TO-92" (id 2) (at 168.91 69.215 0)
       (effects (font (size 1.27 1.27) italic) hide)
     )
@@
     (pin "3")
   )
-  (symbol (lib_id "regulator:XC6206PxxxMR") (at 168.91 96.52 0) (unit 1)
+  (symbol (lib_name "XC6206PxxxMR_1") (lib_id "regulator:XC6206PxxxMR") (at 168.91 96.52 0) (unit 1)
     (in_bom yes) (on_board yes)
     (property "Reference" "URegulator1.2" (id 0) (at 168.91 90.3732 0))
     (property "Value" "1.2V Regulator" (id 1) (at 168.91 92.6846 0))
-    (property "Footprint" "Package_TO_SOT_SMD:SOT-23-3" (id 2) (at 168.91 90.805 0)
+    (property "Footprint" "Package_TO_SOT_THT:TO-92" (id 2) (at 168.91 90.805 0)
       (effects (font (size 1.27 1.27) italic) hide)
     )

Commit message: updated to use new connector footprint
Parts:
- J4: footprint components:camera_connector -> components:CONN_MOLEX_52437-2471
Changed lines of the file:
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@@
       (effects (font (size 1.27 1.27)) (justify left))
     )
-    (property "Footprint" "components:camera_connector" (id 2) (at 91.44 96.52 0)
+    (property "Footprint" "components:CONN_MOLEX_52437-2471" (id 2) (at 91.44 96.52 0)
       (effects (font (size 1.27 1.27)) hide)
     )
