File: Kicad/vogelhuisje_simple/CamMotion/Power_supply.kicad_sch (KiCad schematic)
At the start: 11 parts, among them P1 TP4056breakout, P3 TP4056breakout, P4 TP4056breakout, Q1 Q_PMOS_DGS

Commit message: Finish pcb simplified
Parts:
- D1: renamed from D?; footprint (none) -> Diode_THT:D_A-405_P7.62mm_Horizontal
- P1: footprint Components:TP4056breakout -> components:TP4056breakout
- Rpulldown1: renamed from Rpulldown; footprint (none) -> Resistor_THT:R_Axial_DIN0204_L3.6mm_D1.6mm_P7.62mm_Horizontal
- renumbered UReg to UReg1
Other:
- note added: "Microcontroller input voltage max is lower than output of solar panel"

Commit message: Finished PCB
Now more properly routed
Parts:
- removed Q1: Q_PMOS_DGS, Package_TO_SOT_THT:TO-220-3_Vertical, symbol Device:Q_PMOS_DGS
- added C1: 100u, Capacitor_THT:C_Axial_L5.1mm_D3.1mm_P15.00mm_Horizontal, symbol Device:C
- added C2: 10u, Capacitor_THT:C_Axial_L5.1mm_D3.1mm_P15.00mm_Horizontal, symbol Device:C
- added QPMOS1: TSM680P06CH, Package_TO_SOT_THT:TO-251-3-1EP_Horizontal_TabDown, symbol Device:Q_PMOS_GDS
- UReg1: value LM3940 -> LD1117
Connections:
- net GND: now also C1.2, C2.2
- net Vbat: now also QPMOS1.2 (D)
- net Vcc: now also C1.1, QPMOS1.3 (S)
- net VSolar: now reaches D1.2 (A), JSolar1.2 (Pin_2), P1.1 (Vin+), P3.1 (Vin+), P4.1 (Vin+), Rpulldown1.2
- net VSolar: now also QPMOS1.1 (G)
- net at D1.1 (K), UReg1.1 (VI): now also C2.1
Other:
- moved on the sheet: UReg1
